File: KiCad Files/ttocyobItnA.kicad_sch (KiCad schematic)
At the start: 147 parts, among them J1 ISP, U1 32U4-MU, U2 SRV05-4, Y1 16MHz

Commit message: ああ!
Parts:
- added C10: 100nF, Capacitor_SMD:C_0402_1005Metric, symbol Device:C_Small
- H1, H2, H3, H4, H5, J1, LED1, LED2, MX0-0, MX0-1, MX0-10, MX0-2, MX0-3, MX0-4, MX0-5, MX0-6, MX0-7, MX0-8, MX0-9, MX0-A11, MX0-A12, MX0-B11, MX0-B12, MX1-1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: now left out of the parts list
- renumbered C10 to C11
Connections:
- net +5V: now also C10.1
- net GND: now also C10.2
Other:
- moved on the sheet: C4, C5, C6, C7, C8, C9
